File: project/ZSRing.kicad_pcb (KiCad board)
At the start: 4 copper layers, 0 parts

Commit message: Working on HW revision 1
Parts:
- added C1: 10u, Capacitor_SMD:C_0402_1005Metric, F.Cu at (99.2, 83.2)
- added C10: ~, Capacitor_SMD:C_0201_0603Metric, F.Cu at (58.5, 73.1)
- added C103: 100n, Capacitor_SMD:C_0201_0603Metric, F.Cu at (60.9, 66.1)
- added C104: 4u7, Capacitor_SMD:C_0402_1005Metric, F.Cu at (70.9, 75.3)
- added C105: 100n, Capacitor_SMD:C_0201_0603Metric, F.Cu at (60.9, 67.9)
- added C106: 100p, Capacitor_SMD:C_0201_0603Metric, F.Cu at (60.9, 69.6)
- added C107: 100p, Capacitor_SMD:C_0201_0603Metric, F.Cu at (60.9, 71.4)
- added C108: 100n, Capacitor_SMD:C_0201_0603Metric, F.Cu at (60.9, 73.1)
- added C109: 1u, Capacitor_SMD:C_0201_0603Metric, F.Cu at (60.9, 74.9)
- added C11: ~, Capacitor_SMD:C_0201_0603Metric, F.Cu at (58.5, 74.9)
- added C110: 1u, Capacitor_SMD:C_0201_0603Metric, F.Cu at (60.9, 76.6)
- added C111: 1u, Capacitor_SMD:C_0201_0603Metric, F.Cu at (60.9, 78.4)
- added C112: 10u, Capacitor_SMD:C_0402_1005Metric, F.Cu at (70.9, 77.3)
- added C113: 1u, Capacitor_SMD:C_0201_0603Metric, F.Cu at (63.4, 62.6)
- added C114: 1u, Capacitor_SMD:C_0201_0603Metric, F.Cu at (63.4, 64.4)
- added C115: 12p, Capacitor_SMD:C_0201_0603Metric, F.Cu at (63.4, 66.1)
- added C116: 12p, Capacitor_SMD:C_0201_0603Metric, F.Cu at (63.4, 67.9)
- added C117: 12p, Capacitor_SMD:C_0201_0603Metric, F.Cu at (63.4, 69.6)
- added C118: 12p, Capacitor_SMD:C_0201_0603Metric, F.Cu at (63.4, 71.4)
- added C12: ~, Capacitor_SMD:C_0201_0603Metric, F.Cu at (58.5, 76.6)
- added C13: ~, Capacitor_SMD:C_0201_0603Metric, F.Cu at (58.5, 78.4)
- added C14: ~, Capacitor_SMD:C_0201_0603Metric, F.Cu at (60.9, 62.6)
- added C15: ~, Capacitor_SMD:C_0201_0603Metric, F.Cu at (60.9, 64.4)
- added C16: ~, Capacitor_SMD:C_0201_0603Metric, F.Cu at (82.8, 69.5)
- added C17: ~, Capacitor_SMD:C_0201_0603Metric, F.Cu at (82.8, 71.3)
- added C18: 1u, Capacitor_SMD:C_0201_0603Metric, F.Cu at (82.8, 73.0)
- added C19: 1u8 / 50V, Capacitor_SMD:C_0603_1608Metric, F.Cu at (159.0, 83.9)
- added C2: 10u, Capacitor_SMD:C_0402_1005Metric, F.Cu at (101.2, 81.2)
- added C3: 10u, Capacitor_SMD:C_0402_1005Metric, F.Cu at (103.2, 83.7)
- added C4: 100n, Capacitor_SMD:C_0201_0603Metric, F.Cu at (58.5, 62.6)
- added C5: 100n, Capacitor_SMD:C_0201_0603Metric, F.Cu at (58.5, 64.4)
- added C6: ~, Capacitor_SMD:C_0201_0603Metric, F.Cu at (58.5, 66.1)
- added C7: ~, Capacitor_SMD:C_0201_0603Metric, F.Cu at (58.5, 67.9)
- added C8: 220n / 50V, Capacitor_SMD:C_0603_1608Metric, B.Cu at (159.7, 83.1)
- added C9: 100p / 50V, Capacitor_SMD:C_0603_1608Metric, F.Cu at (58.5, 71.4)
- added D1: STATUS, LED_SMD:LED_0201_0603Metric, B.Cu at (98.3, 81.2)
- added D2: ERROR, LED_SMD:LED_0201_0603Metric, B.Cu at (96.1, 81.2)
- added IC1: nPM1100-CAXX, Package_BGA_Kampi:WLCSP-25_2x2mm_P0.4mm, F.Cu at (101.2, 83.2)
- added IC102: nRF52832-CIXX, Package_BGA_Kampi:WLCSP-56_3x3.2mm_P0.4mm, F.Cu at (111.3, 83.0)
- added IC103: MAX32664, Package_DFN_QFN:QFN-24-1EP_3x3mm_P0.4mm_EP1.75x1.6mm, F.Cu at (75.0, 71.1)
- added IC3: BQ51003YFPR, Package_BGA:Texas_DSBGA-28_1.9x3.0mm_Layout4x7_P0.4mm, B.Cu at (160.0, 86.8)
- added L1: 2u2, Inductor_SMD:L_0201_0603Metric, F.Cu at (102.9, 82.8)
- added L2: ~, pcb_coils:COIL, F.Cu at (165.7, 83.9)
- added Q1: PMZ550UNEYL, Package_SOT_SMD:SOT-883, B.Cu at (96.2, 79.8)
- added Q2: PMZ550UNEYL, Package_SOT_SMD:SOT-883, B.Cu at (98.4, 79.8)
- added Q3: PMZ550UNEYL, Package_SOT_SMD:SOT-883, F.Cu at (105.6, 76.5)
- added Q4: PMZ950UPELYL, Package_SOT_SMD:SOT-883, F.Cu at (106.8, 75.3)
- added R1: 4k7, Resistor_SMD:R_0201_0603Metric, F.Cu at (101.1, 85.0)
- added R10: 10k, Resistor_SMD:R_0201_0603Metric, B.Cu at (97.6, 79.8)
- added R101: 10R, Resistor_SMD:R_0201_0603Metric, F.Cu at (68.3, 67.9)
- added R102: 4k7, Resistor_SMD:R_0201_0603Metric, F.Cu at (68.3, 69.6)
- added R103: 4k7, Resistor_SMD:R_0201_0603Metric, F.Cu at (68.3, 71.4)
- added R104: 4k7, Resistor_SMD:R_0201_0603Metric, F.Cu at (68.3, 73.1)
- added R105: 4k7, Resistor_SMD:R_0201_0603Metric, F.Cu at (68.3, 74.9)
- added R106: 4k7, Resistor_SMD:R_0201_0603Metric, F.Cu at (68.3, 76.6)
- added R11: 10k, Resistor_SMD:R_0201_0603Metric, B.Cu at (95.4, 79.8)
- added R12: 10k, Resistor_SMD:R_0201_0603Metric, F.Cu at (105.6, 75.0)
- added R13: ~, Resistor_SMD:R_0201_0603Metric, F.Cu at (106.8, 76.1)
- added R14: ~, Resistor_SMD:R_0201_0603Metric, F.Cu at (106.8, 76.8)
- added R15: 1k8, Resistor_SMD:R_0201_0603Metric, F.Cu at (68.3, 64.4)
- added R16: 1k8, Resistor_SMD:R_0201_0603Metric, F.Cu at (68.3, 66.1)
- added R2: 10k, Resistor_SMD:R_0201_0603Metric, F.Cu at (100.4, 85.0)
- added R3: ~, Resistor_SMD:R_0201_0603Metric, F.Cu at (63.4, 78.4)
- added R4: ~, Resistor_SMD:R_0201_0603Metric, F.Cu at (65.8, 62.6)
- added R5: ~, Resistor_SMD:R_0201_0603Metric, F.Cu at (65.8, 64.4)
- added R6: ~, Resistor_SMD:R_0201_0603Metric, F.Cu at (65.8, 66.1)
- added R7: ~, Resistor_SMD:R_0201_0603Metric, F.Cu at (65.8, 67.9)
- added R8: 2k, Resistor_SMD:R_0201_0603Metric, B.Cu at (97.6, 81.2)
- added R9: 2k, Resistor_SMD:R_0201_0603Metric, B.Cu at (95.4, 81.2)
- added Y1: 32kHz, Crystal_Kampi:ECS_ECX-1210, F.Cu at (85.2, 69.7)
- added Y101: 32kHz, Crystal:Crystal_SMD_3215-2Pin_3.2x1.5mm, F.Cu at (72.0, 63.4)
- added Y102: 32kHz, Crystal_Kampi:ECS_ECX-1210, F.Cu at (72.0, 66.8)
- added Y103: 32MHz, Crystal_Kampi:Diodes_US, F.Cu at (109.9, 80.2)
Routing:
- net Net-(C10-Pad2): track 0.00 -> 1.70 mm
- net Net-(D2-K): track 0.00 -> 0.72 mm
- net Net-(D1-K): track 0.00 -> 0.72 mm
- net Net-(D2-A): track 0.00 -> 0.70 mm
- net Net-(D1-A): track 0.00 -> 0.70 mm
- net /LED-Error: track 0.00 -> 0.58 mm
- net /LED-Status: track 0.00 -> 0.58 mm
Other:
- board outline added: 75 x 10 mm
- copper layers 4 -> 2
