File: project/ZSRing.kicad_sch (KiCad schematic)
At the start: 0 parts

Commit message: Working on HW revision 1
Parts:
- added AE1: Antenna, symbol Device:Antenna
- added C1, C112, C2, C3: 10u, Capacitor_SMD:C_0402_1005Metric, symbol Device:C
- added C10, C11, C12, C13, C14, C15, C16, C17, C6, C7: ~, Capacitor_SMD:C_0201_0603Metric, symbol Device:C
- added C103, C105, C108: 100n, Capacitor_SMD:C_0201_0603Metric, symbol Device:C
- added C104: 4u7, Capacitor_SMD:C_0402_1005Metric, symbol Device:C
- added C106, C107: 100p, Capacitor_SMD:C_0201_0603Metric, symbol Device:C
- added C109, C110, C111, C113, C114, C18: 1u, Capacitor_SMD:C_0201_0603Metric, symbol Device:C
- added C115, C116, C117, C118: 12p, Capacitor_SMD:C_0201_0603Metric, symbol Device:C
- added C19: 1u8 / 50V, Capacitor_SMD:C_0603_1608Metric, symbol Device:C
- added C4, C5: 100n, Capacitor_SMD:C_0201_0603Metric, symbol Device:C_Small
- added C8: 220n / 50V, Capacitor_SMD:C_0603_1608Metric, symbol Device:C
- added C9: 100p / 50V, Capacitor_SMD:C_0603_1608Metric, symbol Device:C
- added D1: STATUS, LED_SMD:LED_0201_0603Metric, symbol Device:LED
- added D2: ERROR, LED_SMD:LED_0201_0603Metric, symbol Device:LED
- added IC1: nPM1100-CAXX, Package_BGA_Kampi:WLCSP-25_2x2mm_P0.4mm, symbol Nordic:nPM1100-CAXX
- added IC102: nRF52832-CIXX, Package_BGA_Kampi:WLCSP-56_3x3.2mm_P0.4mm, symbol Nordic:nRF52832-CIXX
- added IC103: MAX32664, Package_DFN_QFN:QFN-24-1EP_3x3mm_P0.4mm_EP1.75x1.6mm, symbol AnalogDevices_Kampi:MAX32664
- added IC104: MAXM86161, AnalogDevices:MAXM8616, symbol AnalogDevices_Kampi:MAXM86161
- added IC2: KXTJ3-1057, symbol Rohm:KXTJ3-1057
- added IC3: BQ51003YFPR, Package_BGA:Texas_DSBGA-28_1.9x3.0mm_Layout4x7_P0.4mm, symbol TexasInstruments_Kampi:BQ51003YFPR
- added L1: 2u2, Inductor_SMD:L_0201_0603Metric, symbol Device:L
- added L2: ~, pcb_coils:COIL, symbol Device:L
- added L3: ~, symbol Device:L
- added L4: 10u, symbol Device:L
- added L5: 10n, symbol Device:L
- added Q1, Q2, Q3: PMZ550UNEYL, Package_SOT_SMD:SOT-883, symbol Nexperia:PMZ550UNEYL
- added Q4: PMZ950UPELYL, Package_SOT_SMD:SOT-883, symbol Nexperia:PMZ950UPELYL
- added R1, R102, R103, R104, R105, R106: 4k7, Resistor_SMD:R_0201_0603Metric, symbol Device:R
- added R10, R11, R12, R2: 10k, Resistor_SMD:R_0201_0603Metric, symbol Device:R
- added R101: 10R, Resistor_SMD:R_0201_0603Metric, symbol Device:R
- added R13, R14, R3, R4, R5, R6, R7: ~, Resistor_SMD:R_0201_0603Metric, symbol Device:R
- added R15, R16: 1k8, Resistor_SMD:R_0201_0603Metric, symbol Device:R
- added R8, R9: 2k, Resistor_SMD:R_0201_0603Metric, symbol Device:R
- added TH1: Thermistor_NTC, symbol Device:Thermistor_NTC
- added Y1, Y102: 32kHz, Crystal_Kampi:ECS_ECX-1210, symbol Device:Crystal
- added Y103: 32MHz, Crystal_Kampi:Diodes_US, symbol Device:Crystal
Connections:
- new net: C14.1, IC1.B1 (VBUS), IC1.B2 (VBUS), IC3.D1 (OUT), IC3.D2 (OUT), IC3.D3 (OUT), IC3.D4 (OUT), R3.1, R7.2
- new net: L4.2, L5.1
- new net: C18.1, IC102.A6 (DEC4), L5.2
- new net: C6.1, IC3.E4 (COMM1)
- new net: C13.2, C19.1, C6.2, C7.2, C8.1, C9.1, IC3.B3 (AC1), IC3.B4 (AC1)
- new net: C108.2, R101.2
- new net: C10.1, IC3.C1 (BOOT2)
- new net: C10.2, C11.2, C12.2, C19.2, C9.2, IC3.B1 (AC2), IC3.B2 (AC2), L2.1
- new net: D1.2 (A), R8.2
- new net: C115.2, IC102.D7 (P0.00/XL1), Y102.1
- new net: C117.2, IC102.B2 (XC1), Y103.1
- new net: IC1.E2 (ICHG), R1.1
- new net: C8.2, L2.2
- new net: C111.1, IC103.12 (VCore)
- new net: C106.1, IC102.C2 (DEC3)
- new net: R3.2, R4.2, R5.2
- new net: C12.1, IC3.E2 (CLAMP2)
- new net: C114.1, IC104.4 (VLDO)
- new net: C2.1, IC1.A3 (DEC)
- new net: AE1.1 (A), C17.1, L3.2
- new net: C16.1, IC102.D1 (ANT), L3.1
- new net: IC103.8 (ClockOut), Y1.1
- new net: IC103.9 (ClockIn), Y1.2
- new net: IC102.B6 (DCC), L4.1
- new net: C118.1, IC102.A1 (XC2), Y103.2
- new net: C15.1, IC3.C2 (RECT), IC3.C3 (RECT), R5.1
- new net: C107.1, IC102.A2 (DEC2)
- new net: C103.1, IC102.B7 (DEC1)
- new net: C116.1, IC102.C7 (P0.01/XL2), Y102.2
- new net: IC3.F1 (TS-CTRL), R7.1, TH1.1
- new net: C11.1, IC3.E1 (COMM2)
- new net: Q3.3 (D), Q4.1 (G), R12.2
- new net: Q4.2 (S), R13.1
- new net: IC3.G1 (ILIM), R4.1
- new net: D2.1 (K), Q1.3 (D)
- new net: D2.2 (A), R9.2
- new net: D1.1 (K), Q2.3 (D)
- new net: C13.1, IC3.E3 (CLAMP1)
- new net: C7.1, IC3.C4 (BOOT1)
- new net: IC103.13 (SDA-Sensor), IC104.1 (SDA), R104.2
- new net: C113.1, IC104.12 (VREF)
- new net: IC103.21 (GPIO), IC104.13 (GPIO)
- new net: IC103.14 (SCL-Sensor), IC104.2 (SCL), R105.2
- new net: IC103.20 (LDO-EN), IC104.3 (LDO-EN)
- new net: IC1.B5 (VOUTB), L1.2
- new net: C1.1, IC1.C1 (VSYS), IC1.C2 (VSYS)
- new net: IC1.E1 (NTC), R2.1
- new net: IC3.F2 (FOD), R6.2
- new net +1V8: C104.1, C105.1, C109.1, C110.1, C3.1, C4.1, C5.2, IC1.A4 (SW), IC102.A7 (VDD), IC102.H7 (VDD), IC103.11 (VDD), IC103.22 (VDD), IC2.10 (VDD), IC2.11 (VDDIO), IC2.3 (VDDIO), IC2.7 (VDD), L1.1, R102.1, R103.1, R104.1, R105.1, R106.1, R15.1, R16.1
- new net Acc-Int: IC102.F4 (P0.11), IC2.5 (INT)
- new net Battery: IC102.C6 (P0.02/AIN0), R13.2, R14.1
- new net Battery-Enable: IC102.F7 (P0.06), Q3.1 (G)
- new net Charge: IC1.E4 (CHG)
- new net Error: IC1.E3 (ERR)
- new net GND: C1.2, C103.2, C104.2, C105.2, C106.2, C107.2, C109.2, C110.2, C111.2, C112.2, C113.2, C114.2, C115.1, C116.2, C117.1, C118.2, C14.2, C15.2, C16.2, C17.2, C18.2, C2.2, C3.2, C4.2, C5.1, IC1.A1 (D-), IC1.A5 (PVSS), IC1.B3 (VOUTBSET1), IC1.B4 (VOUTBSET0), IC1.C3 (VTERMSET), IC1.C4 (AVSS), IC1.C5 (AVSS), IC1.D3 (SHPHLD), IC1.D4 (SHPACT), IC1.D5 (ISET), IC1.E5 (MODE), IC102.C4 (GND), IC102.C5 (GND), IC102.D2 (GND), IC102.E3 (GND), IC102.F5 (GND), IC103.10 (GND), IC103.25 (GND), IC103.7 (GND), IC104.10 (DGND), IC104.11 (AGND), IC104.9 (PGND), IC2.1 (ADDR), IC2.4 (RES), IC2.6 (GND), IC2.8 (GND), IC2.9 (GND), IC3.A1 (PGND), IC3.A2 (PGND), IC3.A3 (PGND), IC3.A4 (PGND), IC3.G4 (AD), Q1.2 (S), Q2.2 (S), Q3.2 (S), R1.2, R10.2, R101.1, R11.2, R14.2, R2.2, R6.1, TH1.2
- new net INT_ACC: IC103.19 (Int-ACC)
- new net INT_HR: IC103.18 (Int-HR), IC104.14 (~{INTB}), R106.2
- new net LED-Error: IC102.F6 (P0.07), Q1.1 (G), R11.1
- new net LED-Status: IC102.G7 (P0.08), Q2.1 (G), R10.1
- new net MFIO: IC103.1 (MFIO)
- new net SCL: IC103.24 (SCL), IC2.12 (SCL), R102.2, R15.2
- new net SDA: IC103.23 (SDA), IC2.2 (SDA), R103.2, R16.2
- new net VBAT: IC1.D1 (VBAT), IC1.D2 (VBAT), Q4.3 (D), R12.1, R8.1, R9.1
- new net V_LED: C112.1, IC104.5 (VLED)
- new net ~{RESET}: C108.1, IC103.6 (~{RESET})
- no-connect marks 0 -> 2
