File: testing/Dev-Board/project/Dev-Board.kicad_sch (KiCad schematic)
At the start: 76 parts, among them IC101 BQ51013B, IC102 MAX32664, IC103 MAX30101, IC104 NPM1100-QDAA-R, IC105 TPS61240, IC106 KXTJ3-1057, Q101 BSS138, Q102 BSH205G2AR, X101 BATTERY, X102 INTERFACE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

Commit message: Add layout for Dev-Board
Parts:
- removed R114: 10k, Resistor_SMD:R_0805_2012Metric, symbol Device:R
- added TH102: Thermistor_NTC, Resistor_SMD:R_0805_2012Metric, symbol Device:Thermistor_NTC
- added TP101: +, TestPoint:TestPoint_Pad_1.0x1.0mm, symbol Connector:TestPoint
- added TP102: -, TestPoint:TestPoint_Pad_1.0x1.0mm, symbol Connector:TestPoint
- JP101, JP102, JP103, JP104, JP105, JP106, JP107, JP108, JP109, JP110, JP111, JP112, JP113, JP114, JP115, JP116, JP117, JP118, JP119: footprint Jumper:SolderJumper-2_P1.3mm_Open_Pad1.0x1.5mm -> Connector_PinHeader_2.54mm:PinHeader_1x02_P2.54mm_Vertical
- renumbered R115 to R114, R116 to R115, R117 to R116
Connections:
- net GND: now also TH102.2, TP102.1
- net V_{BAT}: now also TP101.1
- net at IC104.14 (NTC): now also TH102.1

Commit message: Changes from Jakob
Parts:
- removed JP111: CHARGE, Connector_PinHeader_2.54mm:PinHeader_1x02_P2.54mm_Vertical, symbol Jumper:Jumper_2_Open
- removed JP112: ERROR, Connector_PinHeader_2.54mm:PinHeader_1x02_P2.54mm_Vertical, symbol Jumper:Jumper_2_Open
- C121: value 4u7 -> 2u2; Mfr. No. 08055D475KAT4A -> 08055D225KAT4A; Order No. 581-08055D475KAT4A -> 581-08055D225KAT4A
- R107: value 1k -> 18k; Mfr. No. CR0805-JW-102ELF -> CR0805-JW-182ELF; Order No. 652-CR0805-JW-102ELF -> 652-CR0805-JW-182ELF
- R108: value 1k -> 1k8; Mfr. No. CR0805-JW-102ELF -> CR0805-JW-182ELF; Order No. 652-CR0805-JW-102ELF -> 652-CR0805-JW-182ELF
- X102: footprint Connector_PinSocket_2.54mm:PinSocket_1x15_P2.54mm_Vertical -> Connector_PinHeader_2.54mm:PinHeader_1x21_P2.54mm_Vertical; symbol Connector_Generic:Conn_01x15 -> Connector_Generic:Conn_01x21; Mfr. No. 77311-118-15LF -> 77311-118-21LF; Order No. 649-77311-118-15LF -> 649-77311-118-21LF
Connections:
- net Charge: now also IC104.8 (CHG)
- net Error: now also IC104.10 (ERR)
- net GND: now also X102.21 (Pin_21); no longer IC104.11 (SHPHLD), IC104.6 (SHPACT), X102.15 (Pin_15)
- net V_{BAT}: no longer JP114.1 (A), X102.7 (Pin_7)
- net SCL-Slave: now reaches IC102.14 (SCL-Sensor), IC103.2 (SCL), R108.2
- net SCL-Slave: now also X102.16 (Pin_16)
- net SDA-Slave: now reaches IC102.13 (SDA-Sensor), IC103.3 (SDA), R107.2
- net SDA-Slave: now also X102.15 (Pin_15)
- net V_{SYS}: now reaches C118.1, IC104.16 (VSYS)
- net V_{SYS}: now also JP114.1 (A), X102.7 (Pin_7)
- net EN1: now reaches IC101.10 (EN1)
- net EN1: now also X102.17 (Pin_17)
- net EN2: now reaches IC101.11 (EN2)
- net EN2: now also X102.18 (Pin_18)
- new net SHPACT: IC104.6 (SHPACT), X102.19 (Pin_19)
- new net SHPHLD: IC104.11 (SHPHLD), X102.20 (Pin_20)
- no-connect marks 7 -> 5
